Commit message: Now using xacro

File: urdf/rodney.xacro (robot description, xacro)
@@ -1,8 +1,4 @@
-<?xml version="1.0" ?>
-<!-- =================================================================================== -->
-<!-- |    This document was autogenerated by xacro from rodney.xacro                   | -->
-<!-- |    EDITING THIS FILE BY HAND IS NOT RECOMMENDED                                 | -->
-<!-- =================================================================================== -->
-<robot name="Rodney" xmlns:xacro="http://www.ros.org/wiki/xacro">
+<?xml version="1.0"?>
+<robot xmlns:xacro="http://www.ros.org/wiki/xacro" name="Rodney">
   <material name="blue">
     <color rgba="0 0 0.8 1"/>
@@ -20,4 +16,7 @@
     <color rgba="0.8 0.498 0.196 1"/>
   </material>
+  <xacro:property name="base_x" value="0.340"/>
+  <xacro:property name="base_y" value="0.180"/>
+  <xacro:property name="base_z" value="0.010"/>
   <link name="base_link">
     <visual>
@@ -25,9 +24,9 @@
         <mesh filename="package://rodney/meshes/rodneyBase.dae"/>
       </geometry>
-      <origin xyz="0.0 0.0 -0.005"/>
-    </visual>
-    <collision>
-      <geometry>
-        <box size="0.34 0.18 0.01"/>
+      <origin xyz="0.0 0.0 -${base_z/2.0}"/>
+    </visual>
+    <collision>
+      <geometry>
+        <box size="${base_x} ${base_y} ${base_z}"/>
       </geometry>
     </collision>
@@ -43,5 +42,5 @@
         <box size="0.075 0.056 0.030"/>
       </geometry>
-      <material name="black"/>
+      <material name="black" />
     </visual>
     <collision>
@@ -65,5 +64,5 @@
         <box size="0.146 0.074 0.020"/>
       </geometry>
-      <material name="black"/>
+      <material name="black" />
     </visual>
     <collision>
@@ -158,5 +157,5 @@
     <parent link="left_motor_bracket"/>
     <child link="left_wheel"/>
-    <dynamic damping="200.0" friction="200.0"/>
+    <dynamic damping="200.0" friction="200.0" />
     <origin xyz="0.0 0.029 -0.0105"/>
   </joint>
@@ -236,5 +235,5 @@
     <parent link="right_motor_bracket"/>
     <child link="right_wheel"/>
-    <dynamic damping="200.0" friction="200.0"/>
+    <dynamic damping="200.0" friction="200.0" />
     <origin xyz="0.0 -0.029 -0.0105"/>
   </joint>
@@ -246,5 +245,5 @@
         <box size="0.025 0.040 0.065"/>
       </geometry>
-      <material name="blue"/>
+      <material name="blue" />
     </visual>
     <collision>
@@ -268,5 +267,5 @@
         <sphere radius="0.020"/>
       </geometry>
-      <material name="white"/>
+      <material name="white" />
     </visual>
     <collision>
@@ -292,5 +291,5 @@
         <box size="0.025 0.040 0.065"/>
       </geometry>
-      <material name="blue"/>
+      <material name="blue" />
     </visual>
     <collision>
@@ -314,5 +313,5 @@
         <sphere radius="0.020"/>
       </geometry>
-      <material name="white"/>
+      <material name="white" />
     </visual>
     <collision>
@@ -333,108 +332,39 @@
   </joint>
   <!-- Rear platform -->
-  <link name="rear_post_1">
-    <visual>
-      <geometry>
-        <cylinder length="0.02" radius="0.005"/>
-      </geometry>
-      <origin xyz="0.0 0.0 0.01"/>
-      <material name="blue"/>
-    </visual>
-    <collision>
-      <geometry>
-        <cylinder length="0.02" radius="0.005"/>
-      </geometry>
-      <origin xyz="0.0 0.0 0.01"/>
-    </collision>
-    <inertial>
-      <!-- Move centre of gravity back to middle of link -->
-      <origin xyz="0.0 0.0 0.01"/>
-      <mass value="0.001"/>
-      <inertia ixx="3.95833e-8" ixy="0.0" ixz="0.0" iyy="3.95833e-8" iyz="0.0" izz="1.25e-8"/>
-    </inertial>
-  </link>
-  <joint name="base_to_rear_post_1" type="fixed">
-    <parent link="base_link"/>
-    <child link="rear_post_1"/>
-    <origin xyz="-0.06 0.08 0.005"/>
-  </joint>
-  <link name="rear_post_2">
-    <visual>
-      <geometry>
-        <cylinder length="0.02" radius="0.005"/>
-      </geometry>
-      <origin xyz="0.0 0.0 0.01"/>
-      <material name="blue"/>
-    </visual>
-    <collision>
-      <geometry>
-        <cylinder length="0.02" radius="0.005"/>
-      </geometry>
-      <origin xyz="0.0 0.0 0.01"/>
-    </collision>
-    <inertial>
-      <!-- Move centre of gravity back to middle of link -->
-      <origin xyz="0.0 0.0 0.01"/>
-      <mass value="0.001"/>
-      <inertia ixx="3.95833e-8" ixy="0.0" ixz="0.0" iyy="3.95833e-8" iyz="0.0" izz="1.25e-8"/>
-    </inertial>
-  </link>
-  <joint name="base_to_rear_post_2" type="fixed">
-    <parent link="base_link"/>
-    <child link="rear_post_2"/>
-    <origin xyz="-0.14 0.08 0.005"/>
-  </joint>
-  <link name="rear_post_3">
-    <visual>
-      <geometry>
-        <cylinder length="0.02" radius="0.005"/>
-      </geometry>
-      <origin xyz="0.0 0.0 0.01"/>
-      <material name="blue"/>
-    </visual>
-    <collision>
-      <geometry>
-        <cylinder length="0.02" radius="0.005"/>
-      </geometry>
-      <origin xyz="0.0 0.0 0.01"/>
-    </collision>
-    <inertial>
-      <!-- Move centre of gravity back to middle of link -->
-      <origin xyz="0.0 0.0 0.01"/>
-      <mass value="0.001"/>
-      <inertia ixx="3.95833e-8" ixy="0.0" ixz="0.0" iyy="3.95833e-8" iyz="0.0" izz="1.25e-8"/>
-    </inertial>
-  </link>
-  <joint name="base_to_rear_post_3" type="fixed">
-    <parent link="base_link"/>
-    <child link="rear_post_3"/>
-    <origin xyz="-0.06 -0.08 0.005"/>
-  </joint>
-  <link name="rear_post_4">
-    <visual>
-      <geometry>
-        <cylinder length="0.02" radius="0.005"/>
-      </geometry>
-      <origin xyz="0.0 0.0 0.01"/>
-      <material name="blue"/>
-    </visual>
-    <collision>
-      <geometry>
-        <cylinder length="0.02" radius="0.005"/>
-      </geometry>
-      <origin xyz="0.0 0.0 0.01"/>
-    </collision>
-    <inertial>
-      <!-- Move centre of gravity back to middle of link -->
-      <origin xyz="0.0 0.0 0.01"/>
-      <mass value="0.001"/>
-      <inertia ixx="3.95833e-8" ixy="0.0" ixz="0.0" iyy="3.95833e-8" iyz="0.0" izz="1.25e-8"/>
-    </inertial>
-  </link>
-  <joint name="base_to_rear_post_4" type="fixed">
-    <parent link="base_link"/>
-    <child link="rear_post_4"/>
-    <origin xyz="-0.14 -0.08 0.005"/>
-  </joint>
+  <xacro:property name="rear_post_height" value="0.020"/>
+  <xacro:property name="rear_post_radius" value="0.005"/>
+  <xacro:macro name="rear_post" params="postfix pos_x reflect_y">
+    <link name="rear_post_${postfix}">
+      <visual>
+        <geometry>
+          <cylinder length="${rear_post_height}" radius="${rear_post_radius}"/>
+        </geometry>
+        <origin xyz="0.0 0.0 ${rear_post_height/2.0}"/>
+        <material name="blue"/>
+      </visual>
+      <collision>
+        <geometry>
+          <cylinder length="${rear_post_height}" radius="${rear_post_radius}"/>
+        </geometry>
+        <origin xyz="0.0 0.0 ${rear_post_height/2.0}"/>
+      </collision>
+      <inertial>
+        <!-- Move centre of gravity back to middle of link -->
+        <origin xyz="0.0 0.0 ${rear_post_height/2.0}"/>
+        <mass value="0.001"/>
+        <inertia ixx="3.95833e-8" ixy="0.0" ixz="0.0" iyy="3.95833e-8" iyz="0.0" izz="1.25e-8"/>
+      </inertial>
+    </link>
+    <joint name="base_to_rear_post_${postfix}" type="fixed">
+      <parent link="base_link"/>
+      <child link="rear_post_${postfix}"/>
+      <origin xyz="${pos_x} ${reflect_y*((base_y/2.0)-0.010)} ${base_z/2.0}"/>
+    </joint>
+  </xacro:macro>
+  <xacro:rear_post postfix="1" pos_x="-0.06" reflect_y="1"/>
+  <xacro:rear_post postfix="2" pos_x="-0.14" reflect_y="1"/>
+  <xacro:rear_post postfix="3" pos_x="-0.06" reflect_y="-1"/>
+  <xacro:rear_post postfix="4" pos_x="-0.14" reflect_y="-1"/>
+  <xacro:property name="rear_platf_z" value="0.003"/>
   <link name="rear_platform">
     <visual>
@@ -442,5 +372,5 @@
         <mesh filename="package://rodney/meshes/smallRearPlatform.dae"/>
       </geometry>
-      <origin rpy="0 0 1.57" xyz="0.050 0.0 -0.0015"/>
+      <origin rpy="0 0 1.57" xyz="0.050 0.0 -${rear_platf_z/2.0}"/>
     </visual>
     <collision>
@@ -457,5 +387,5 @@
     <parent link="rear_post_1"/>
     <child link="rear_platform"/>
-    <origin xyz="-0.040 -0.080 0.0215"/>
+    <origin xyz="-0.040 -0.080 ${rear_post_height+(rear_platf_z/2.0)}"/>
   </joint>
   <!-- Neck and head -->
@@ -644,108 +574,39 @@
   </joint>
   <!-- Front platform -->
-  <link name="fwd_post_1">
-    <visual>
-      <geometry>
-        <cylinder length="0.055" radius="0.005"/>
-      </geometry>
-      <origin xyz="0.0 0.0 0.0275"/>
-      <material name="blue"/>
-    </visual>
-    <collision>
-      <geometry>
-        <cylinder length="0.055" radius="0.005"/>
-      </geometry>
-      <origin xyz="0.0 0.0 0.0275"/>
-    </collision>
-    <inertial>
-      <!-- Move centre of gravity back to middle of link -->
-      <origin xyz="0.0 0.0 0.0275"/>
-      <mass value="0.0015"/>
-      <inertia ixx="1.12594e-7" ixy="0.0" ixz="0.0" iyy="1.12594e-7" iyz="0.0" izz="1.875e-10"/>
-    </inertial>
-  </link>
-  <joint name="base_to_fwd_post_1" type="fixed">
-    <parent link="base_link"/>
-    <child link="fwd_post_1"/>
-    <origin xyz="0.14 0.08 0.005"/>
-  </joint>
-  <link name="fwd_post_2">
-    <visual>
-      <geometry>
-        <cylinder length="0.055" radius="0.005"/>
-      </geometry>
-      <origin xyz="0.0 0.0 0.0275"/>
-      <material name="blue"/>
-    </visual>
-    <collision>
-      <geometry>
-        <cylinder length="0.055" radius="0.005"/>
-      </geometry>
-      <origin xyz="0.0 0.0 0.0275"/>
-    </collision>
-    <inertial>
-      <!-- Move centre of gravity back to middle of link -->
-      <origin xyz="0.0 0.0 0.0275"/>
-      <mass value="0.0015"/>
-      <inertia ixx="1.12594e-7" ixy="0.0" ixz="0.0" iyy="1.12594e-7" iyz="0.0" izz="1.875e-10"/>
-    </inertial>
-  </link>
-  <joint name="base_to_fwd_post_2" type="fixed">
-    <parent link="base_link"/>
-    <child link="fwd_post_2"/>
-    <origin xyz="0.14 -0.08 0.005"/>
-  </joint>
-  <link name="fwd_post_3">
-    <visual>
-      <geometry>
-        <cylinder length="0.055" radius="0.005"/>
-      </geometry>
-      <origin xyz="0.0 0.0 0.0275"/>
-      <material name="blue"/>
-    </visual>
-    <collision>
-      <geometry>
-        <cylinder length="0.055" radius="0.005"/>
-      </geometry>
-      <origin xyz="0.0 0.0 0.0275"/>
-    </collision>
-    <inertial>
-      <!-- Move centre of gravity back to middle of link -->
-      <origin xyz="0.0 0.0 0.0275"/>
-      <mass value="0.0015"/>
-      <inertia ixx="1.12594e-7" ixy="0.0" ixz="0.0" iyy="1.12594e-7" iyz="0.0" izz="1.875e-10"/>
-    </inertial>
-  </link>
-  <joint name="base_to_fwd_post_3" type="fixed">
-    <parent link="base_link"/>
-    <child link="fwd_post_3"/>
-    <origin xyz="0.085 -0.08 0.005"/>
-  </joint>
-  <link name="fwd_post_4">
-    <visual>
-      <geometry>
-        <cylinder length="0.055" radius="0.005"/>
-      </geometry>
-      <origin xyz="0.0 0.0 0.0275"/>
-      <material name="blue"/>
-    </visual>
-    <collision>
-      <geometry>
-        <cylinder length="0.055" radius="0.005"/>
-      </geometry>
-      <origin xyz="0.0 0.0 0.0275"/>
-    </collision>
-    <inertial>
-      <!-- Move centre of gravity back to middle of link -->
-      <origin xyz="0.0 0.0 0.0275"/>
-      <mass value="0.0015"/>
-      <inertia ixx="1.12594e-7" ixy="0.0" ixz="0.0" iyy="1.12594e-7" iyz="0.0" izz="1.875e-10"/>
-    </inertial>
-  </link>
-  <joint name="base_to_fwd_post_4" type="fixed">
-    <parent link="base_link"/>
-    <child link="fwd_post_4"/>
-    <origin xyz="0.085 0.08 0.005"/>
-  </joint>
+  <xacro:property name="fwd_post_height" value="0.055"/>
+  <xacro:property name="fwd_post_radius" value="0.005"/>
+  <xacro:macro name="fwd_post" params="postfix pos_x reflect_y">
+    <link name="fwd_post_${postfix}">
+      <visual>
+        <geometry>
+          <cylinder length="${fwd_post_height}" radius="${fwd_post_radius}"/>
+        </geometry>
+        <origin xyz="0.0 0.0 ${fwd_post_height/2.0}"/>
+        <material name="blue"/>
+      </visual>
+      <collision>
+        <geometry>
+          <cylinder length="${fwd_post_height}" radius="${fwd_post_radius}"/>
+        </geometry>
+        <origin xyz="0.0 0.0 ${fwd_post_height/2.0}"/>
+      </collision>
+      <inertial>
+        <!-- Move centre of gravity back to middle of link -->
+        <origin xyz="0.0 0.0 ${fwd_post_height/2.0}"/>
+        <mass value="0.0015"/>
+        <inertia ixx="1.12594e-7" ixy="0.0" ixz="0.0" iyy="1.12594e-7" iyz="0.0" izz="1.875e-10"/>
+      </inertial>
+    </link>
+    <joint name="base_to_fwd_post_${postfix}" type="fixed">
+      <parent link="base_link"/>
+      <child link="fwd_post_${postfix}"/>
+      <origin xyz="${pos_x} ${reflect_y*((base_y/2.0)-0.010)} ${base_z/2.0}"/>
+    </joint>
+  </xacro:macro>
+  <xacro:fwd_post postfix="1" pos_x="0.14" reflect_y="1"/>
+  <xacro:fwd_post postfix="2" pos_x="0.14" reflect_y="-1"/>
+  <xacro:fwd_post postfix="3" pos_x="0.085" reflect_y="-1"/>
+  <xacro:fwd_post postfix="4" pos_x="0.085" reflect_y="1"/>
+  <xacro:property name="fwd_platf_z" value="0.003"/>
   <link name="fwd_platform">
     <visual>
@@ -762,5 +623,5 @@
     <inertial>
       <mass value="0.030"/>
-      <inertia ixx="8.1e-5" ixy="0.0" ixz="0.0" iyy="4.02e-6" iyz="0.0" izz="0.000085"/>
+      <inertia ixx="8.1e-5" ixy="0.0" ixz="0.0" iyy="4.02e-6" iyz="0.0" izz="0.000085" />
     </inertial>
   </link>
@@ -768,5 +629,5 @@
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
Commit message: updates to xacro

File: urdf/rodney.xacro (robot description, xacro)
@@ -631,7 +631,7 @@
     <origin xyz="-0.040 -0.080 ${fwd_post_height+(fwd_platf_z/2.0)}"/>
   </joint>
-  <!-- LIDAR link -->
+  <!-- LIDAR -->
   <!-- Using mesh of a model -->
-  <link name="lidar_link">
+  <link name="laser">
     <visual>
       <geometry>
@@ -679,5 +679,5 @@
     <origin xyz="0.0 0.0 0.0175"/>
   </joint>
-  <link name="lidar_link">
+  <link name="laser">
     <visual>
       <geometry>
@@ -857,5 +857,5 @@
   </gazebo>
   <!-- LIDAR -->
-  <gazebo reference="lidar_link">
+  <gazebo reference="laser">
     <sensor type="ray" name="base_lidar_sensor">
       <pose>0 0 0 0 0 0</pose>
@@ -884,5 +884,5 @@
       <plugin name="gazebo_ros_head_hokuyo_controller" filename="libgazebo_ros_laser.so">
         <topicName>scan</topicName>
-        <frameName>lidar_link</frameName>
+        <frameName>laser</frameName>
       </plugin>
     </sensor>
