Commit message: More modelling

File: urdf/rodney.urdf (robot description, URDF)
Before this commit: robot Rodney, 21 links, 20 joints
Links:
- added link head_pan_bracket; visual mesh filename=package://rodney/meshes/headPanBracket.dae
- added link head_tilt_arm; visual mesh filename=package://rodney/meshes/headTiltArm.dae
Joints:
- added joint head_pan_bracket_to_head_tilt_arm: type revolute, parent head_pan_bracket, child head_tilt_arm, origin xyz=0.0 -0.01 0.035 rpy=0 0 0, axis 0 1 0, limit lower=-1.572 upper=0.3 effort=1000.0 velocity=0.5
- added joint servo_block_to_head_pan_bracket: type revolute, parent head_pan_servo_block, child head_pan_bracket, origin xyz=0.01 0.0 0.037 rpy=0 0 3.142, axis 0 0 1, limit lower=-1.571 upper=1.571 effort=1000.0 velocity=0.5

Commit message: Added screen to model

File: urdf/rodney.urdf (robot description, URDF)
Before this commit: robot Rodney, 23 links, 22 joints
Links:
- added link display; visual box size=0.005 0.192 0.110
- added link display_bracket; visual mesh filename=package://rodney/meshes/displayBracket.dae
Joints:
- added joint display_bracket_to_display: type fixed, parent display_bracket, child display, origin xyz=0.0025 0.0 0.06 rpy=0 0 0
- added joint head_tilt_arm_to_display_bracket: type fixed, parent head_tilt_arm, child display_bracket, origin xyz=0.059 0.008 0.0 rpy=0 0 0

Commit message: Thinking a bit more about the model transforms

File: urdf/rodney.urdf (robot description, URDF)
Before this commit: robot Rodney, 25 links, 24 joints
Links:
- link head_pan_servo_block: geometry visual box size=0.057 0.032 0.066
Joints:
- joint base_to_fl_motor_brk: origin xyz=0.075 0.091 -0.0245 rpy=1.58 0 0 -> xyz=0.075 0.091 0.0
- joint base_to_fr_motor_brk: origin xyz=0.075 -0.091 -0.0245 rpy=1.58 0 0 -> xyz=0.075 -0.091 0.0
- joint base_to_post_1: origin xyz=-0.06 0.08 0.033 -> xyz=-0.06 0.08 0.008
- joint base_to_post_2: origin xyz=-0.14 0.08 0.033 -> xyz=-0.14 0.08 0.008
- joint base_to_post_3: origin xyz=-0.06 -0.08 0.033 -> xyz=-0.06 -0.08 0.008
- joint base_to_post_4: origin xyz=-0.14 -0.08 0.033 -> xyz=-0.14 -0.08 0.008
- joint base_to_rl_motor_brk: origin xyz=-0.075 0.091 -0.0245 rpy=1.58 0 0 -> xyz=-0.075 0.091 0.0
- joint base_to_rr_motor_brk: origin xyz=-0.075 -0.091 -0.0245 rpy=1.58 0 0 -> xyz=-0.075 -0.091 0.0
- joint display_bracket_to_display: origin xyz=0.0025 0.0 0.06 rpy=0 0 0 -> xyz=0.003 0.008 0.060
- joint fl_brk_to_fl_motor: origin xyz=0.0 -0.0055 0.028 rpy=0 0 0 -> xyz=0.0 -0.001 -0.028
- joint fl_brk_to_wheel: axis 0 0 1 -> 0 1 0; origin xyz=0.0 -0.0055 -0.025 rpy=0 0 0 -> xyz=0.0 0.001 -0.034
- joint fr_brk_to_fr_motor: origin xyz=0.0 -0.0055 -0.028 rpy=0 0 0 -> xyz=0.0 0.001 -0.028
- joint fr_brk_to_wheel: axis 0 0 1 -> 0 1 0; origin xyz=0.0 -0.0055 0.025 rpy=0 0 0 -> xyz=0.0 -0.001 -0.034
- joint head_fixing_to_servo_block: origin xyz=-0.010 0.0 0.084 rpy=0 0 0 -> xyz=0.0 0.0 0.047
- joint head_pan_bracket_to_head_tilt_arm: origin xyz=0.0 -0.01 0.035 rpy=0 0 0 -> xyz=0.0 -0.009 0.035
- joint head_tilt_arm_to_display_bracket: origin xyz=0.059 0.008 0.0 rpy=0 0 0 -> xyz=0.056 0.0 0.0
- joint neck_to_head_fixing: origin xyz=0.0 0.0 0.112 rpy=0 0 1.58 -> xyz=0.0 0.0 0.30
- joint post_1_to_rear_platform: origin xyz=0.01 -0.08 0.025 rpy=0 0 1.58 -> xyz=0.0 0.0 0.05
- joint rear_platform_to_neck: origin xyz=0 0.08 0.1 -> xyz=-0.070 -0.080 -0.050
- joint rl_brk_to_rl_motor: origin xyz=0.0 -0.0055 0.028 rpy=0 0 0 -> xyz=0.0 -0.001 -0.028
- joint rl_brk_to_wheel: axis 0 0 1 -> 0 1 0; origin xyz=0.0 -0.0055 -0.025 rpy=0 0 0 -> xyz=0.0 0.001 -0.034
- joint rr_brk_to_rr_motor: origin xyz=0.0 -0.0055 -0.028 rpy=0 0 0 -> xyz=0.0 0.001 -0.028
- joint rr_brk_to_wheel: axis 0 0 1 -> 0 1 0; origin xyz=0.0 -0.0055 0.025 rpy=0 0 0 -> xyz=0.0 -0.001 -0.028
- joint servo_block_to_head_pan_bracket: origin xyz=0.01 0.0 0.037 rpy=0 0 3.142 -> xyz=0.0 0.0 0.025

Commit message: mass and inertia added

File: urdf/rodney.urdf (robot description, URDF)
Before this commit: robot Rodney, 25 links, 24 joints
Links:
- link base_link: mass None -> 1; geometry collision box size=0.340 0.180 0.008; visual mesh filename=package://rodney/meshes/rodneyBase.dae
- link display: mass None -> 1.0; geometry collision box size=0.005 0.192 0.110; visual box size=0.005 0.192 0.110
- link display_bracket: mass None -> 0.020; geometry collision box size=0.010 0.146 0.045; visual mesh filename=package://rodney/meshes/displayBracket.dae
- link front_left_motor: mass None -> 0.198; geometry collision cylinder length=0.056 radius=0.0185; visual cylinder length=0.056 radius=0.0185
- link front_left_motor_bracket: mass None -> 0.035; geometry collision box size=0.042 0.049 0.002; visual box size=0.042 0.049 0.002
- link front_left_wheel: mass None -> 0.105; geometry collision cylinder length=0.050 radius=0.053; visual cylinder length=0.050 radius=0.053
- link front_right_motor: mass None -> 0.198; geometry collision cylinder length=0.056 radius=0.0185; visual cylinder length=0.056 radius=0.0185
- link front_right_motor_bracket: mass None -> 0.035; geometry collision box size=0.042 0.049 0.002; visual box size=0.042 0.049 0.002
- link front_right_wheel: mass None -> 0.105; geometry collision cylinder length=0.050 radius=0.053; visual cylinder length=0.050 radius=0.053
- link head_fixing: mass None -> 0.015; geometry collision box size=0.03 0.04 0.1; visual mesh filename=package://rodney/meshes/headFixing.dae
- link head_pan_bracket: mass None -> 0.020; geometry collision box size=0.025 0.068 0.045; visual mesh filename=package://rodney/meshes/headPanBracket.dae
- link head_pan_servo_block: mass None -> 0.015; geometry collision box size=0.057 0.032 0.066; visual box size=0.057 0.032 0.066
- link head_tilt_arm: mass None -> 0.020; geometry collision box size=0.075 0.065 0.020; visual mesh filename=package://rodney/meshes/headTiltArm.dae
- link neck: mass None -> 0.030; geometry collision cylinder length=0.30 radius=0.011; visual cylinder length=0.30 radius=0.011
- link post_1: mass None -> 0.009; geometry collision cylinder length=0.05 radius=0.005; visual cylinder length=0.05 radius=0.005
- link post_2: mass None -> 0.009; geometry collision cylinder length=0.05 radius=0.005; visual cylinder length=0.05 radius=0.005
- link post_3: mass None -> 0.009; geometry collision cylinder length=0.05 radius=0.005; visual cylinder length=0.05 radius=0.005
- link post_4: mass None -> 0.009; geometry collision cylinder length=0.05 radius=0.005; visual cylinder length=0.05 radius=0.005
- link rear_left_motor: mass None -> 0.198; geometry collision cylinder length=0.056 radius=0.0185; visual cylinder length=0.056 radius=0.0185
- link rear_left_motor_bracket: mass None -> 0.035; geometry collision box size=0.042 0.049 0.002; visual box size=0.042 0.049 0.002
- link rear_left_wheel: mass None -> 0.105; geometry collision cylinder length=0.050 radius=0.053; visual cylinder length=0.050 radius=0.053
- link rear_platform: mass None -> 0.061; geometry collision box size=0.180 0.098 0.003; visual mesh filename=package://rodney/meshes/smallRearPlatform.dae
- link rear_right_motor: mass None -> 0.198; geometry collision cylinder length=0.056 radius=0.0185; visual cylinder length=0.056 radius=0.0185
- link rear_right_motor_bracket: mass None -> 0.035; geometry collision box size=0.042 0.049 0.002; visual box size=0.042 0.049 0.002
- link rear_right_wheel: mass None -> 0.105; geometry collision cylinder length=0.050 radius=0.053; visual cylinder length=0.050 radius=0.053

Commit message: Using the model in gazebo

File: urdf/rodney.urdf (robot description, URDF)
Before this commit: robot Rodney, 25 links, 24 joints
Links:
- link base_link: mass 1 -> 2
- link display: mass 1.0 -> 0.010

Commit message: Updated mass values

File: urdf/rodney.urdf (robot description, URDF)
Before this commit: robot Rodney, 25 links, 24 joints
Links:
- link base_link: mass 2 -> 0.297
- link display: mass 0.010 -> 0.338
- link display_bracket: mass 0.020 -> 0.012
- link front_left_motor: mass 0.198 -> 0.196
- link front_left_wheel: mass 0.105 -> 0.117
- link front_right_motor: mass 0.198 -> 0.196
- link front_right_wheel: mass 0.105 -> 0.117
- link head_pan_bracket: mass 0.020 -> 0.010
- link head_pan_servo_block: mass 0.015 -> 0.084
- link head_tilt_arm: mass 0.020 -> 0.019
- link neck: mass 0.030 -> 0.033
- link post_1: mass 0.009 -> 0.001
- link post_2: mass 0.009 -> 0.001
- link post_3: mass 0.009 -> 0.001
- link post_4: mass 0.009 -> 0.001
- link rear_left_motor: mass 0.198 -> 0.196
- link rear_left_wheel: mass 0.105 -> 0.117
- link rear_platform: mass 0.061 -> 0.050
- link rear_right_motor: mass 0.198 -> 0.196
- link rear_right_wheel: mass 0.105 -> 0.117

Commit message: More model work

File: urdf/rodney.urdf (robot description, URDF)
Before this commit: robot Rodney, 25 links, 24 joints
Links:
- added link AAx10, mass 0.259; collision box size=0.075 0.056 0.030; visual box size=0.075 0.056 0.030
- added link USB_PACK, mass 0.358; collision box size=0.146 0.074 0.020; visual box size=0.146 0.074 0.020
- link display: mass 0.338 -> 0.010
- link post_1: geometry collision cylinder length=0.020 radius=0.005; visual cylinder length=0.020 radius=0.005
- link post_2: geometry collision cylinder length=0.020 radius=0.005; visual cylinder length=0.020 radius=0.005
- link post_3: geometry collision cylinder length=0.020 radius=0.005; visual cylinder length=0.020 radius=0.005
- link post_4: geometry collision cylinder length=0.020 radius=0.005; visual cylinder length=0.020 radius=0.005
Joints:
- added joint base_to_AAx10: type fixed, parent base_link, child AAx10, origin xyz=0.0 0.0 0.0
- added joint base_to_USB_PACK: type fixed, parent base_link, child USB_PACK, origin xyz=0.010 0.0 0.008
- joint base_to_fl_motor_brk: origin xyz=0.075 0.091 0.0 -> xyz=0.075 0.095 0.0
- joint base_to_fr_motor_brk: origin xyz=0.075 -0.091 0.0 -> xyz=0.075 -0.095 0.0
- joint base_to_rl_motor_brk: origin xyz=-0.075 0.091 0.0 -> xyz=-0.075 0.095 0.0
- joint base_to_rr_motor_brk: origin xyz=-0.075 -0.091 0.0 -> xyz=-0.075 -0.095 0.0
- joint post_1_to_rear_platform: origin xyz=0.0 0.0 0.05 -> xyz=0.0 0.0 0.02
- joint rear_platform_to_neck: origin xyz=-0.070 -0.080 -0.050 -> xyz=-0.070 -0.080 -0.028

Commit message: Changed from 4WD to 2WD

File: urdf/rodney.urdf (robot description, URDF)
Before this commit: robot Rodney, 27 links, 26 joints
Links:
- removed link front_left_motor
- removed link front_left_motor_bracket
- removed link front_left_wheel
- removed link front_right_motor
- removed link front_right_motor_bracket
- removed link front_right_wheel
- removed link rear_left_motor
- removed link rear_left_motor_bracket
- removed link rear_left_wheel
- removed link rear_right_motor
- removed link rear_right_motor_bracket
- removed link rear_right_wheel
- added link front_caster, mass 0.003; collision sphere radius=0.020; visual sphere radius=0.020
- added link front_caster_bracket, mass 0.030; collision box size=.025 0.040 0.060; visual box size=0.025 0.040 0.060
- added link left_motor, mass 0.196; collision cylinder length=0.056 radius=0.0185; visual cylinder length=0.056 radius=0.0185
- added link left_motor_bracket, mass 0.035; collision box size=0.042 0.049 0.002; visual box size=0.042 0.049 0.002
- added link left_wheel, mass 0.117; collision cylinder length=0.050 radius=0.053; visual cylinder length=0.050 radius=0.053
- added link rear_caster, mass 0.003; collision sphere radius=0.020; visual sphere radius=0.020
- added link rear_caster_bracket, mass 0.030; collision box size=.025 0.040 0.060; visual box size=0.025 0.040 0.060
- added link right_motor, mass 0.196; collision cylinder length=0.056 radius=0.0185; visual cylinder length=0.056 radius=0.0185
- added link right_motor_bracket, mass 0.035; collision box size=0.042 0.049 0.002; visual box size=0.042 0.049 0.002
- added link right_wheel, mass 0.117; collision cylinder length=0.050 radius=0.053; visual cylinder length=0.050 radius=0.053
Joints:
- removed joint base_to_fl_motor_brk
- removed joint base_to_fr_motor_brk
- removed joint base_to_rl_motor_brk
- removed joint base_to_rr_motor_brk
- removed joint fl_brk_to_fl_motor
- removed joint fl_brk_to_wheel
- removed joint fr_brk_to_fr_motor
- removed joint fr_brk_to_wheel
- removed joint rl_brk_to_rl_motor
- removed joint rl_brk_to_wheel
- removed joint rr_brk_to_rr_motor
- removed joint rr_brk_to_wheel
- added joint base_to_front_caster: type fixed, parent base_link, child front_caster_bracket, origin xyz=0.150 0.0 -0.060
- added joint base_to_l_motor_brk: type fixed, parent base_link, child left_motor_bracket, origin xyz=0.0 0.095 0.0
- added joint base_to_r_motor_brk: type fixed, parent base_link, child right_motor_bracket, origin xyz=0.0 -0.095 0.0
- added joint base_to_rear_caster: type fixed, parent base_link, child rear_caster_bracket, origin xyz=-0.150 0.0 -0.060
- added joint front_caster_bk_to_ball: type continuous, parent front_caster_bracket, child front_caster, origin xyz=0.0 0.0 0.0, axis 1 1 1
- added joint l_brk_to_l_motor: type fixed, parent left_motor_bracket, child left_motor, origin xyz=0.0 -0.001 -0.028
- added joint l_brk_to_wheel: type continuous, parent left_motor_bracket, child left_wheel, origin xyz=0.0 0.001 -0.034, axis 0 1 0
- added joint r_brk_to_r_motor: type fixed, parent right_motor_bracket, child right_motor, origin xyz=0.0 0.001 -0.028
- added joint r_brk_to_wheel: type continuous, parent right_motor_bracket, child right_wheel, origin xyz=0.0 -0.001 -0.034, axis 0 1 0
- added joint rear_caster_bk_to_ball: type continuous, parent rear_caster_bracket, child rear_caster, origin xyz=0.0 0.0 0.0, axis 1 1 1
- joint base_to_AAx10: origin xyz=0.0 0.0 0.0 -> xyz=0.060 0.0 0.0
- joint base_to_USB_PACK: origin xyz=0.010 0.0 0.008 -> xyz=0.060 0.0 0.008

Commit message: Fixing controllers

File: urdf/rodney.urdf (robot description, URDF)
Before this commit: robot Rodney, 25 links, 24 joints
Links:
- link display: mass 0.010 -> 0.338

Commit message: Changes so rviz follows real robot head

File: urdf/rodney.urdf (robot description, URDF)
Before this commit: robot Rodney, 25 links, 24 joints
Joints:
- joint head_pan_bracket_to_head_tilt_arm: limit lower=-1.572 upper=0.3 effort=1000.0 velocity=0.5 -> lower=-1.396 upper=0.698 effort=1000.0 velocity=0.5

Commit message: Changed names of head joints in model

File: urdf/rodney.urdf (robot description, URDF)
Before this commit: robot Rodney, 25 links, 24 joints
Joints:
- removed joint head_pan_bracket_to_head_tilt_arm
- removed joint servo_block_to_head_pan_bracket
- added joint head_pan: type revolute, parent head_pan_servo_block, child head_pan_bracket, origin xyz=0.0 0.0 0.025, axis 0 0 1, limit lower=-1.5708 upper=1.5708 effort=1000.0 velocity=0.5
- added joint head_tilt: type revolute, parent head_pan_bracket, child head_tilt_arm, origin xyz=0.0 -0.009 0.035, axis 0 1 0, limit lower=-1.39626 upper=0.698132 effort=1000.0 velocity=0.5

Commit message: Code tidy

File: urdf/rodney.urdf (robot description, URDF)
Before this commit: robot Rodney, 25 links, 24 joints
Links:
- link front_caster_bracket: geometry collision box size=.025 0.040 0.070; visual box size=0.025 0.040 0.070
- link left_motor: mass 0.196 -> 0.206; geometry collision cylinder length=0.070 radius=0.0185; visual cylinder length=0.070 radius=0.0185
- link rear_caster_bracket: geometry collision box size=.025 0.040 0.070; visual box size=0.025 0.040 0.070
- link right_motor: mass 0.196 -> 0.206; geometry collision cylinder length=0.070 radius=0.0185; visual cylinder length=0.070 radius=0.0185
Joints:
- joint base_to_front_caster: origin xyz=0.150 0.0 -0.060 -> xyz=0.150 0.0 -0.070
- joint base_to_rear_caster: origin xyz=-0.150 0.0 -0.060 -> xyz=-0.150 0.0 -0.070
- joint front_caster_bk_to_ball: origin xyz=0.0 0.0 0.0 -> xyz=0.0 0.0 0.004
- joint rear_caster_bk_to_ball: origin xyz=0.0 0.0 0.0 -> xyz=0.0 0.0 0.004

Commit message: Added a camera to the model

File: urdf/rodney.urdf (robot description, URDF)
Before this commit: robot Rodney, 25 links, 24 joints
Links:
- added link camera, mass 1e-5; collision box size=0.005 0.025 0.020; visual box size=0.005 0.025 0.020
Joints:
- added joint camera_joint: type fixed, parent display, child camera, origin xyz=0.0 0.0 0.065

Commit message: Added LIDAR to URDF model

File: urdf/rodney.urdf (robot description, URDF)
Before this commit: robot Rodney, 26 links, 25 joints
Links:
- added link fwd_platform, mass 0.030; collision box size=0.04 0.018 0.003; visual box size=0.04 0.18 0.003
- added link fwd_post_1, mass 0.0015; collision cylinder length=0.030 radius=0.005; visual cylinder length=0.030 radius=0.005
- added link fwd_post_2, mass 0.0015; collision cylinder length=0.030 radius=0.005; visual cylinder length=0.030 radius=0.005
- added link fwd_post_3, mass 0.0015; collision cylinder length=0.030 radius=0.005; visual cylinder length=0.030 radius=0.005
- added link fwd_post_4, mass 0.0015; collision cylinder length=0.030 radius=0.005; visual cylinder length=0.030 radius=0.005
- added link lidar_link, mass 1e-5; collision box size=0.02 0.03 0.01; visual box size=0.02 0.03 0.01
Joints:
- added joint base_to_fwd_post_1: type fixed, parent base_link, child fwd_post_1, origin xyz=0.14 0.08 0.008
- added joint base_to_fwd_post_2: type fixed, parent base_link, child fwd_post_2, origin xyz=0.14 -0.08 0.008
- added joint base_to_fwd_post_3: type fixed, parent base_link, child fwd_post_3, origin xyz=0.12 -0.08 0.008
- added joint base_to_fwd_post_4: type fixed, parent base_link, child fwd_post_4, origin xyz=0.12 0.08 0.008
- added joint fwd_post_1_to_fwd_platform: type fixed, parent fwd_post_1, child fwd_platform, origin xyz=-0.01 -0.08 0.030
- added joint lidar_to_fwd_platform: type fixed, parent fwd_platform, child lidar_link, origin xyz=0.0 0.0 0.0065

Commit message: Added fwd platform mesh

File: urdf/rodney.urdf (robot description, URDF)
Before this commit: robot Rodney, 32 links, 31 joints
Links:
- added link lidar_servo, mass 0.084; collision box size=0.041 0.020 0.040; visual box size=0.041 0.020 0.040
- link fwd_platform: geometry collision box size=0.075 0.018 0.003; visual mesh filename=package://rodney/meshes/fwdPlatform.dae
- link fwd_post_1: geometry collision cylinder length=0.055 radius=0.005; visual cylinder length=0.055 radius=0.005
- link fwd_post_2: geometry collision cylinder length=0.055 radius=0.005; visual cylinder length=0.055 radius=0.005
- link fwd_post_3: geometry collision cylinder length=0.055 radius=0.005; visual cylinder length=0.055 radius=0.005
- link fwd_post_4: geometry collision cylinder length=0.055 radius=0.005; visual cylinder length=0.055 radius=0.005
- link lidar_link: geometry collision box size=0.040 0.048 0.020; visual box size=0.040 0.048 0.020
Joints:
- removed joint lidar_to_fwd_platform
- added joint fwd_platform_to_lidar_servo: type fixed, parent fwd_platform, child lidar_servo, origin xyz=0.010 0.0 -0.007
- added joint lidar_to_lidar_servo: type fixed, parent lidar_servo, child lidar_link, origin xyz=0.020 0.0 0.030
- joint base_to_fwd_post_3: origin xyz=0.12 -0.08 0.008 -> xyz=0.085 -0.08 0.008
- joint base_to_fwd_post_4: origin xyz=0.12 0.08 0.008 -> xyz=0.085 0.08 0.008
- joint fwd_post_1_to_fwd_platform: origin xyz=-0.01 -0.08 0.030 -> xyz=-0.0275 -0.080 0.055

Commit message: changes to urdf model

File: urdf/rodney.urdf (robot description, URDF)
Before this commit: robot Rodney, 33 links, 32 joints
Links:
- link display: mass 0.338 -> 0.0

Commit message: Changes to model

File: urdf/rodney.urdf (robot description, URDF)
Before this commit: robot Rodney, 33 links, 32 joints
Links:
- removed link lidar_servo
- link base_link: geometry collision box size=0.340 0.180 0.010; visual mesh filename=package://rodney/meshes/rodneyBase.dae
- link front_caster_bracket: geometry collision box size=0.025 0.040 0.065; visual box size=0.025 0.040 0.065
- link left_wheel: geometry collision cylinder length=0.050 radius=0.050; visual cylinder length=0.050 radius=0.050
- link lidar_link: mass 1e-5 -> 0.213; geometry collision box size=0.0985 0.070 0.060; visual mesh filename=package://rodney/meshes/rplidar.dae
- link rear_caster_bracket: geometry collision box size=0.025 0.040 0.065; visual box size=0.025 0.040 0.065
- link right_wheel: geometry collision cylinder length=0.050 radius=0.050; visual cylinder length=0.050 radius=0.050
Joints:
- removed joint fwd_platform_to_lidar_servo
- removed joint lidar_to_lidar_servo
- added joint fwd_platform_to_lidar: type fixed, parent fwd_platform, child lidar_link, origin xyz=-0.015 0.0 0.0455
- joint base_to_AAx10: origin xyz=0.060 0.0 0.0 -> xyz=0.070 0.0 -0.020
- joint base_to_USB_PACK: origin xyz=0.060 0.0 0.008 -> xyz=0.060 0.0 0.015
- joint base_to_front_caster: origin xyz=0.150 0.0 -0.070 -> xyz=0.150 0.0 -0.0375
- joint base_to_fwd_post_1: origin xyz=0.14 0.08 0.008 -> xyz=0.14 0.08 0.0325
- joint base_to_fwd_post_2: origin xyz=0.14 -0.08 0.008 -> xyz=0.14 -0.08 0.0325
- joint base_to_fwd_post_3: origin xyz=0.085 -0.08 0.008 -> xyz=0.085 -0.08 0.0325
- joint base_to_fwd_post_4: origin xyz=0.085 0.08 0.008 -> xyz=0.085 0.08 0.0325
- joint base_to_l_motor_brk: origin xyz=0.0 0.095 0.0 -> xyz=0.0 0.091 -0.0295
- joint base_to_post_1: origin xyz=-0.06 0.08 0.008 -> xyz=-0.06 0.08 0.015
- joint base_to_post_2: origin xyz=-0.14 0.08 0.008 -> xyz=-0.14 0.08 0.015
- joint base_to_post_3: origin xyz=-0.06 -0.08 0.008 -> xyz=-0.06 -0.08 0.015
- joint base_to_post_4: origin xyz=-0.14 -0.08 0.008 -> xyz=-0.14 -0.08 0.015
- joint base_to_r_motor_brk: origin xyz=0.0 -0.095 0.0 -> xyz=0.0 -0.091 -0.0295
- joint base_to_rear_caster: origin xyz=-0.150 0.0 -0.070 -> xyz=-0.150 0.0 -0.0375
- joint display_bracket_to_display: origin xyz=0.003 0.008 0.060 -> xyz=0.0055 0.008 0.060
- joint front_caster_bk_to_ball: origin xyz=0.0 0.0 0.004 -> xyz=0.0 0.0 -0.0315
- joint fwd_post_1_to_fwd_platform: origin xyz=-0.0275 -0.080 0.055 -> xyz=-0.040 -0.080 0.029
- joint head_fixing_to_servo_block: origin xyz=0.0 0.0 0.047 -> xyz=0.008 0.0 0.039
- joint head_pan: origin xyz=0.0 0.0 0.025 -> xyz=-0.008 0.0 0.033
- joint l_brk_to_l_motor: origin xyz=0.0 -0.001 -0.028 -> xyz=0.0 -0.036 -0.004
- joint l_brk_to_wheel: origin xyz=0.0 0.001 -0.034 -> xyz=0.0 0.029 -0.0105
- joint neck_to_head_fixing: origin xyz=0.0 0.0 0.30 -> xyz=0.0 0.0 0.150
- joint post_1_to_rear_platform: origin xyz=0.0 0.0 0.02 -> xyz=-0.040 -0.080 0.0115
- joint r_brk_to_r_motor: origin xyz=0.0 0.001 -0.028 -> xyz=0.0 0.036 -0.004
- joint r_brk_to_wheel: origin xyz=0.0 -0.001 -0.034 -> xyz=0.0 -0.029 -0.0105
- joint rear_caster_bk_to_ball: origin xyz=0.0 0.0 0.004 -> xyz=0.0 0.0 -0.0315
- joint rear_platform_to_neck: origin xyz=-0.070 -0.080 -0.028 -> xyz=-0.030 0.0 0.1205
