Commit message: Changes to moments of inertia

File: urdf/rodney.urdf (robot description, URDF)
Before this commit: robot Rodney, 32 links, 31 joints
Links:
- link base_link: mass 0.297 -> 0.300
- link camera: mass 1e-5 -> 0.001
Joints:
- joint front_caster_bk_to_ball: origin xyz=0.0 0.0 -0.0315 -> xyz=0.0 0.0 -0.0325
- joint head_tilt: limit lower=-1.39626 upper=0.698132 effort=1000.0 velocity=0.5 -> lower=-1.39626 upper=0.5 effort=1000.0 velocity=0.698132
- joint rear_caster_bk_to_ball: origin xyz=0.0 0.0 -0.0315 -> xyz=0.0 0.0 -0.0325

Commit message: fixed gravity model problem

File: urdf/rodney.urdf (robot description, URDF)
Before this commit: robot Rodney, 32 links, 31 joints
Links:
- link display: mass 0.0 -> 0.338

Commit message: development

File: urdf/rodney.urdf (robot description, URDF)
Before this commit: robot Rodney, 32 links, 31 joints
Links:
- removed link lidar_link
- added link laser, mass 0.213; collision box size=0.0985 0.070 0.060; visual mesh filename=package://rodney/meshes/rplidar.dae
Joints:
- removed joint base_to_l_motor_brk
- removed joint base_to_r_motor_brk
- removed joint l_brk_to_l_motor
- removed joint l_brk_to_wheel
- removed joint r_brk_to_r_motor
- removed joint r_brk_to_wheel
- added joint base_to_left_motor_bracket: type fixed, parent base_link, child left_motor_bracket, origin xyz=0.0 0.091 -0.0291
- added joint base_to_right_motor_bracket: type fixed, parent base_link, child right_motor_bracket, origin xyz=0.0 -0.091 -0.0291
- added joint left_brk_to_left_motor: type fixed, parent left_motor_bracket, child left_motor, origin xyz=0.0 -0.036 -0.004
- added joint left_brk_to_left_wheel: type continuous, parent left_motor_bracket, child left_wheel, origin xyz=0.0 0.029 -0.0105
- added joint right_brk_to_right_motor: type fixed, parent right_motor_bracket, child right_motor, origin xyz=0.0 0.036 -0.004
- added joint right_brk_to_right_wheel: type continuous, parent right_motor_bracket, child right_wheel, origin xyz=0.0 -0.029 -0.0105
- joint base_to_front_caster: origin xyz=0.150 0.0 -0.0375 -> xyz=0.15 0.0 -0.0375
- joint base_to_rear_caster: origin xyz=-0.150 0.0 -0.0375 -> xyz=-0.15 0.0 -0.0375
- joint fwd_platform_to_lidar: child lidar_link -> laser

File: urdf/rodney.xacro (robot description, xacro)
@@ -82,253 +82,149 @@
   </joint>
   <!-- Motors and wheels -->
+  <xacro:macro name="motor_bracket" params="prefix reflect">
+    <link name="${prefix}_motor_bracket">
+      <visual>
+        <geometry>
+          <box size="0.042 0.049 0.002"/>
+        </geometry>
+        <origin rpy="1.58 0 0"/>
+        <material name="bronze"/>
+      </visual>
+      <collision>
+        <geometry>
+          <box size="0.042 0.049 0.002"/>
+        </geometry>
+        <origin rpy="1.58 0 0"/>
+      </collision>
+      <inertial>
+        <origin rpy="1.58 0 0"/>
+        <mass value="0.035"/>
+        <inertia ixx="7.01e-6" ixy="0.0" ixz="0.0" iyy="5.16e-6" iyz="0.0" izz="1.21e-5"/>
+      </inertial>
+    </link>
+    <joint name="base_to_${prefix}_motor_bracket" type="fixed">
+      <parent link="base_link"/>
+      <child link="${prefix}_motor_bracket"/>
+      <origin xyz="0.0 ${reflect*0.091} -0.0291"/>
+    </joint>
+  </xacro:macro>
+  <xacro:macro name="motor" params="prefix reflect">
+    <link name="${prefix}_motor">
+      <visual>
+        <geometry>
+          <cylinder length="0.070" radius="0.0185"/>
+        </geometry>
+        <origin rpy="1.57 0 0"/>
+        <material name="silver"/>
+      </visual>
+      <collision>
+        <geometry>
+          <cylinder length="0.070" radius="0.0185"/>
+        </geometry>
+        <origin rpy="1.57 0 0"/>
+      </collision>
+      <inertial>
+        <origin rpy="1.57 0 0"/>
+        <mass value="0.206"/>
+        <inertia ixx="0.000101743" ixy="0.0" ixz="0.0" iyy="0.000101743" iyz="0.0" izz="3.52518e-5"/>
+      </inertial>
+    </link>
+    <joint name="${prefix}_brk_to_${prefix}_motor" type="fixed">
+      <parent link="${prefix}_motor_bracket"/>
+      <child link="${prefix}_motor"/>
+      <origin xyz="0.0 ${reflect*0.036} -0.004"/>
+    </joint>
+  </xacro:macro>
+  <xacro:macro name="wheel" params="prefix reflect">
+    <link name="${prefix}_wheel">
+      <visual>
+        <geometry>
+          <cylinder length="0.050" radius="0.050"/>
+        </geometry>
+        <origin rpy="1.57 0 0"/>
+        <material name="black"/>
+      </visual>
+      <collision>
+        <geometry>
+          <cylinder length="0.050" radius="0.050"/>
+        </geometry>
+        <origin rpy="1.57 0 0"/>
+      </collision>
+      <inertial>
+        <origin rpy="1.57 0 0"/>
+        <mass value="0.117"/>
+      <inertia ixx="0.0000975" ixy="0.0" ixz="0.0" iyy="0.0000975" iyz="0.0" izz="0.00014625"/>
+      </inertial>
+    </link>
+    <joint name="${prefix}_brk_to_${prefix}_wheel" type="continuous">
+      <parent link="${prefix}_motor_bracket"/>
+      <child link="${prefix}_wheel"/>
+      <origin xyz="0.0 ${reflect*0.029} -0.0105"/>
+    </joint>
+  </xacro:macro>
   <!-- left -->
-  <link name="left_motor_bracket">
-    <visual>
-      <geometry>
-        <box size="0.042 0.049 0.002"/>
-      </geometry>
-      <origin rpy="1.58 0 0"/>
-      <material name="bronze"/>
-    </visual>
-    <collision>
-      <geometry>
-        <box size="0.042 0.049 0.002"/>
-      </geometry>
-      <origin rpy="1.58 0 0"/>
-    </collision>
-    <inertial>
-      <origin rpy="1.58 0 0"/>
-      <mass value="0.035"/>
-      <inertia ixx="7.01e-6" ixy="0.0" ixz="0.0" iyy="5.16e-6" iyz="0.0" izz="1.21e-5"/>
-    </inertial>
-  </link>
-  <joint name="base_to_l_motor_brk" type="fixed">
-    <parent link="base_link"/>
-    <child link="left_motor_bracket"/>
-    <origin xyz="0.0 0.091 -0.0295"/>
-  </joint>
-  <link name="left_motor">
-    <visual>
-      <geometry>
-        <cylinder length="0.070" radius="0.0185"/>
-      </geometry>
-      <origin rpy="1.57 0 0"/>
-      <material name="silver"/>
-    </visual>
-    <collision>
-      <geometry>
-        <cylinder length="0.070" radius="0.0185"/>
-      </geometry>
-      <origin rpy="1.57 0 0"/>
-    </collision>
-    <inertial>
-      <origin rpy="1.57 0 0"/>
-      <mass value="0.206"/>
-      <inertia ixx="0.000101743" ixy="0.0" ixz="0.0" iyy="0.000101743" iyz="0.0" izz="3.52518e-5"/>
-    </inertial>
-  </link>
-  <joint name="l_brk_to_l_motor" type="fixed">
-    <parent link="left_motor_bracket"/>
-    <child link="left_motor"/>
-    <origin xyz="0.0 -0.036 -0.004"/>
-  </joint>
-  <link name="left_wheel">
-    <visual>
-      <geometry>
-        <cylinder length="0.050" radius="0.050"/>
-      </geometry>
-      <origin rpy="1.57 0 0"/>
-      <material name="black"/>
-    </visual>
-    <collision>
-      <geometry>
-        <cylinder length="0.050" radius="0.050"/>
-      </geometry>
-      <origin rpy="1.57 0 0"/>
-    </collision>
-    <inertial>
-      <origin rpy="1.57 0 0"/>
-      <mass value="0.117"/>
-      <inertia ixx="0.0000975" ixy="0.0" ixz="0.0" iyy="0.0000975" iyz="0.0" izz="0.00014625"/>
-    </inertial>
-  </link>
-  <joint name="l_brk_to_wheel" type="continuous">
-    <axis xyz="0 1 0"/>
-    <parent link="left_motor_bracket"/>
-    <child link="left_wheel"/>
-    <dynamic damping="200.0" friction="200.0" />
-    <origin xyz="0.0 0.029 -0.0105"/>
-  </joint>
+  <xacro:motor_bracket prefix="left" reflect="1"/>
+  <xacro:motor prefix="left" reflect="-1"/>
+  <xacro:wheel prefix="left" reflect="1"/>
   <!-- right -->
-  <link name="right_motor_bracket">
-    <visual>
-      <geometry>
-        <box size="0.042 0.049 0.002"/>
-      </geometry>
-      <origin rpy="1.58 0 0"/>
-      <material name="bronze"/>
-    </visual>
-    <collision>
-      <geometry>
-        <box size="0.042 0.049 0.002"/>
-      </geometry>
-      <origin rpy="1.58 0 0"/>
-    </collision>
-    <inertial>
-      <origin rpy="1.58 0 0"/>
-      <mass value="0.035"/>
-      <inertia ixx="7.01e-6" ixy="0.0" ixz="0.0" iyy="5.16e-6" iyz="0.0" izz="1.21e-5"/>
-    </inertial>
-  </link>
-  <joint name="base_to_r_motor_brk" type="fixed">
-    <parent link="base_link"/>
-    <child link="right_motor_bracket"/>
-    <origin xyz="0.0 -0.091 -0.0295"/>
-  </joint>
-  <link name="right_motor">
-    <visual>
-      <geometry>
-        <cylinder length="0.070" radius="0.0185"/>
-      </geometry>
-      <origin rpy="1.57 0 0"/>
-      <material name="silver"/>
-    </visual>
-    <collision>
-      <geometry>
-        <cylinder length="0.070" radius="0.0185"/>
-      </geometry>
-      <origin rpy="1.57 0 0"/>
-    </collision>
-    <inertial>
-      <origin rpy="1.57 0 0"/>
-      <mass value="0.206"/>
-      <inertia ixx="0.000101743" ixy="0.0" ixz="0.0" iyy="0.000101743" iyz="0.0" izz="3.52518e-5"/>
-    </inertial>
-  </link>
-  <joint name="r_brk_to_r_motor" type="fixed">
-    <parent link="right_motor_bracket"/>
-    <child link="right_motor"/>
-    <origin xyz="0.0 0.036 -0.004"/>
-  </joint>
-  <link name="right_wheel">
-    <visual>
-      <geometry>
-        <cylinder length="0.050" radius="0.050"/>
-      </geometry>
-      <origin rpy="1.57 0 0"/>
-      <material name="black"/>
-    </visual>
-    <collision>
-      <geometry>
-        <cylinder length="0.050" radius="0.050"/>
-      </geometry>
-      <origin rpy="1.57 0 0"/>
-    </collision>
-    <inertial>
-      <origin rpy="1.57 0 0"/>
-      <mass value="0.117"/>
-      <inertia ixx="0.0000975" ixy="0.0" ixz="0.0" iyy="0.0000975" iyz="0.0" izz="0.00014625"/>
-    </inertial>
-  </link>
-  <joint name="r_brk_to_wheel" type="continuous">
-    <axis xyz="0 1 0"/>
-    <parent link="right_motor_bracket"/>
-    <child link="right_wheel"/>
-    <dynamic damping="200.0" friction="200.0" />
-    <origin xyz="0.0 -0.029 -0.0105"/>
-  </joint>
+  <xacro:motor_bracket prefix="right" reflect="-1"/>
+  <xacro:motor prefix="right" reflect="1"/>
+  <xacro:wheel prefix="right" reflect="-1"/>
   <!-- Casters -->
+  <xacro:macro name="caster_bracket" params="prefix reflect">
+    <link name="${prefix}_caster_bracket">
+      <visual>
+        <geometry>
+          <box size="0.025 0.040 0.065"/>
+        </geometry>
+        <material name="blue" />
+      </visual>
+      <collision>
+        <geometry>
+          <box size="0.025 0.040 0.065"/>
+        </geometry>
+      </collision>
+      <inertial>
+        <mass value="0.030"/>
+        <inertia ixx="1.46e-5" ixy="0.0" ixz="0.0" iyy="2.21e-5" iyz="0.0" izz="5.56e-6"/>
+      </inertial>
+    </link>
+    <joint name="base_to_${prefix}_caster" type="fixed">
+      <parent link="base_link"/>
+      <child link="${prefix}_caster_bracket"/>
+      <origin xyz="${reflect*0.150} 0.0 -0.0375"/>
+    </joint>
+  </xacro:macro>
+  <xacro:macro name="caster" params="prefix">
+    <link name="${prefix}_caster">
+      <visual>
+        <geometry>
+          <sphere radius="0.020"/>
+        </geometry>
+        <material name="white" />
+      </visual>
+      <collision>
+        <geometry>
+          <sphere radius="0.020"/>
+        </geometry>
+      </collision>
+      <inertial>
+        <mass value="0.003"/>
+        <inertia ixx="4.8e-7" ixy="0.0" ixz="0.0" iyy="4.8e-7" iyz="0.0" izz="4.8e-7"/>
+      </inertial>
+    </link>
+    <joint name="${prefix}_caster_bk_to_ball" type="continuous">
+      <axis xyz="1 1 1"/>
+      <parent link="${prefix}_caster_bracket"/>
+      <child link="${prefix}_caster"/>
+      <origin xyz="0.0 0.0 -0.0325"/>
+    </joint>
+  </xacro:macro>
   <!-- Front -->
-  <link name="front_caster_bracket">
-    <visual>
-      <geometry>
-        <box size="0.025 0.040 0.065"/>
-      </geometry>
-      <material name="blue" />
-    </visual>
-    <collision>
-      <geometry>
-        <box size="0.025 0.040 0.065"/>
-      </geometry>
-    </collision>
-    <inertial>
-      <mass value="0.030"/>
-      <inertia ixx="1.46e-5" ixy="0.0" ixz="0.0" iyy="2.21e-5" iyz="0.0" izz="5.56e-6"/>
-    </inertial>
-  </link>
-  <joint name="base_to_front_caster" type="fixed">
-    <parent link="base_link"/>
-    <child link="front_caster_bracket"/>
-    <origin xyz="0.150 0.0 -0.0375"/>
-  </joint>
-  <link name="front_caster">
-    <visual>
-      <geometry>
-        <sphere radius="0.020"/>
-      </geometry>
-      <material name="white" />
-    </visual>
-    <collision>
-      <geometry>
-        <sphere radius="0.020"/>
-      </geometry>
-    </collision>
-    <inertial>
-      <mass value="0.003"/>
-      <inertia ixx="4.8e-7" ixy="0.0" ixz="0.0" iyy="4.8e-7" iyz="0.0" izz="4.8e-7"/>
-    </inertial>
-  </link>
-  <joint name="front_caster_bk_to_ball" type="continuous">
-    <axis xyz="1 1 1"/>
-    <parent link="front_caster_bracket"/>
-    <child link="front_caster"/>
-    <origin xyz="0.0 0.0 -0.0325"/>
-  </joint>
+  <xacro:caster_bracket prefix="front" reflect="1"/>
+  <xacro:caster prefix="front"/>
   <!-- Rear -->
-  <link name="rear_caster_bracket">
-    <visual>
-      <geometry>
-        <box size="0.025 0.040 0.065"/>
-      </geometry>
-      <material name="blue" />
-    </visual>
-    <collision>
-      <geometry>
-        <box size="0.025 0.040 0.065"/>
-      </geometry>
-    </collision>
-    <inertial>
-      <mass value="0.030"/>
-      <inertia ixx="1.46e-5" ixy="0.0" ixz="0.0" iyy="2.21e-5" iyz="0.0" izz="5.56e-6"/>
-    </inertial>
-  </link>
-  <joint name="base_to_rear_caster" type="fixed">
-    <parent link="base_link"/>
-    <child link="rear_caster_bracket"/>
-    <origin xyz="-0.150 0.0 -0.0375"/>
-  </joint>
-  <link name="rear_caster">
-    <visual>
-      <geometry>
-        <sphere radius="0.020"/>
-      </geometry>
-      <material name="white" />
-    </visual>
-    <collision>
-      <geometry>
-        <sphere radius="0.020"/>
-      </geometry>
-    </collision>
-    <inertial>
-      <mass value="0.003"/>
-      <inertia ixx="4.8e-7" ixy="0.0" ixz="0.0" iyy="4.8e-7" iyz="0.0" izz="4.8e-7"/>
-    </inertial>
-  </link>
-  <joint name="rear_caster_bk_to_ball" type="continuous">
-    <axis xyz="1 1 1"/>
-    <parent link="rear_caster_bracket"/>
-    <child link="rear_caster"/>
-    <origin xyz="0.0 0.0 -0.0325"/>
-  </joint>
+  <xacro:caster_bracket prefix="rear" reflect="-1"/>
+  <xacro:caster prefix="rear"/>
   <!-- Rear platform -->
   <xacro:property name="rear_post_height" value="0.020"/>
@@ -652,5 +548,5 @@
   <joint name="fwd_platform_to_lidar" type="fixed">
     <parent link="fwd_platform"/>
-    <child link ="lidar_link"/>
+    <child link ="laser"/>
     <origin xyz="-0.015 0.0 0.0455"/>
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
Commit message: Fixing fault introduced

File: urdf/rodney.urdf (robot description, URDF)
Before this commit: robot Rodney, 32 links, 31 joints
Joints:
- joint base_to_front_caster: origin xyz=0.15 0.0 -0.0375 -> xyz=0.15 0.0 -0.037
- joint base_to_rear_caster: origin xyz=-0.15 0.0 -0.0375 -> xyz=-0.15 0.0 -0.037
- joint left_brk_to_left_wheel: axis (none) -> 0 1 0
- joint right_brk_to_right_wheel: axis (none) -> 0 1 0

File: urdf/rodney.xacro (robot description, xacro)
@@ -158,4 +158,5 @@
     </link>
     <joint name="${prefix}_brk_to_${prefix}_wheel" type="continuous">
+      <axis xyz="0 1 0"/>
       <parent link="${prefix}_motor_bracket"/>
       <child link="${prefix}_wheel"/>
@@ -193,5 +194,5 @@
       <parent link="base_link"/>
       <child link="${prefix}_caster_bracket"/>
-      <origin xyz="${reflect*0.150} 0.0 -0.0375"/>
+      <origin xyz="${reflect*0.150} 0.0 -0.037"/>
     </joint>
   </xacro:macro>
@@ -605,14 +606,14 @@
     <material>Gazebo/Black</material>
   </gazebo>
-  <gazebo reference="post_1">
-    <material>Gazebo/Blue</material>
-  </gazebo>
-  <gazebo reference="post_2">
-    <material>Gazebo/Blue</material>
-  </gazebo>
-  <gazebo reference="post_3">
-    <material>Gazebo/Blue</material>
-  </gazebo>
-  <gazebo reference="post_4">
+  <gazebo reference="rear_post_1">
+    <material>Gazebo/Blue</material>
+  </gazebo>
+  <gazebo reference="rear_post_2">
+    <material>Gazebo/Blue</material>
+  </gazebo>
+  <gazebo reference="rear_post_3">
+    <material>Gazebo/Blue</material>
+  </gazebo>
+  <gazebo reference="rear_post_4">
     <material>Gazebo/Blue</material>
   </gazebo>
@@ -671,6 +672,6 @@
       <wheelAcceleration>0</wheelAcceleration>
       <wheelTorque>5</wheelTorque>
-      <leftJoint>l_brk_to_wheel</leftJoint>
-      <rightJoint>r_brk_to_wheel</rightJoint>
+      <leftJoint>left_brk_to_left_wheel</leftJoint>
+      <rightJoint>right_brk_to_right_wheel</rightJoint>
       <wheelSeparation>0.230</wheelSeparation>
       <wheelDiameter>0.106</wheelDiameter>
@@ -683,8 +684,7 @@
   <!-- To control head pan/tilt -->
   <gazebo>
-    <plugin name="gazebo_ros_control" filename="libgazebo_ros_control.so"/>
-    <robotNamespace>/Rodney</robotNamespace>
-    <robotSimType>gazebo_ros_control/DefaultRobotHWSim</robotSimType>
-    <legacyModeNS>True</legacyModeNS>
+    <plugin name="gazebo_ros_control" filename="libgazebo_ros_control.so">
+      <legacyModeNS>true</legacyModeNS>
+    </plugin>
   </gazebo>
   <transmission name="head_pan_tran">
@@ -711,5 +711,5 @@
     <plugin name="joint_state_publisher"
             filename="libgazebo_ros_joint_state_publisher.so">
-      <jointName>head_pan, head_tilt, front_caster_bk_to_ball, rear_caster_bk_to_ball, l_brk_to_wheel, r_brk_to_wheel</jointName>
+      <jointName>head_pan, head_tilt, front_caster_bk_to_ball, rear_caster_bk_to_ball, left_brk_to_left_wheel, right_brk_to_right_wheel</jointName>
       <updateRate>20.0</updateRate>
     </plugin>
