Commit message: Adding lidar (#9)
* Added LIDAR to URDF model

* Update to use Teensy

* LIDAR servo min range set and onboard LED turned on

* Added fwd platform mesh

* added origin to each inertial tag where it is not the default

* Changes for LIDAR sweep

* More LIDAR changes

* changes to urdf model

* No LIDAR but can configure for Teensy or Arduino Nano

* Conditional compile for Arduino Nano or Teensy

* Launch file updated for Teensy to use 500000 baud rate

* Moving scripts to own folder

* Increased tacho publish rate to 40Hz on a Teensy

* Changes to model

* Changes to moments of inertia

* fixed gravity model problem

* Now using xacro

* updates to xacro

* development

* Fixing fault introduced

* development or using nav stack

* More nav development

* Removed old maps

* Planning plugins merged into LIDAR branch (#8)

* Looking at different planner plugins

* Adding in EKF to fuse odom and IMU

* More development

* Update package.xml

* Update CHANGELOG.rst

* Still looking at improving nav

* Change in nav parameters

* Update to node documentation

File: urdf/rodney.urdf (robot description, URDF)
Before this commit: robot Rodney, 26 links, 25 joints
Links:
- removed link post_1
- removed link post_2
- removed link post_3
- removed link post_4
- added link fwd_platform, mass 0.030; collision box size=0.075 0.018 0.003; visual mesh filename=package://rodney/meshes/fwdPlatform.dae
- added link fwd_post_1, mass 0.0015; collision cylinder length=0.055 radius=0.005; visual cylinder length=0.055 radius=0.005
- added link fwd_post_2, mass 0.0015; collision cylinder length=0.055 radius=0.005; visual cylinder length=0.055 radius=0.005
- added link fwd_post_3, mass 0.0015; collision cylinder length=0.055 radius=0.005; visual cylinder length=0.055 radius=0.005
- added link fwd_post_4, mass 0.0015; collision cylinder length=0.055 radius=0.005; visual cylinder length=0.055 radius=0.005
- added link laser, mass 0.213; collision box size=0.0985 0.070 0.060; visual mesh filename=package://rodney/meshes/rplidar.dae
- added link rear_post_1, mass 0.001; collision cylinder length=0.02 radius=0.005; visual cylinder length=0.02 radius=0.005
- added link rear_post_2, mass 0.001; collision cylinder length=0.02 radius=0.005; visual cylinder length=0.02 radius=0.005
- added link rear_post_3, mass 0.001; collision cylinder length=0.02 radius=0.005; visual cylinder length=0.02 radius=0.005
- added link rear_post_4, mass 0.001; collision cylinder length=0.02 radius=0.005; visual cylinder length=0.02 radius=0.005
- link base_link: mass 0.297 -> 0.300; geometry collision box size=0.34 0.18 0.01; visual mesh filename=package://rodney/meshes/rodneyBase.dae
- link camera: mass 1e-5 -> 0.001
- link front_caster_bracket: geometry collision box size=0.025 0.040 0.065; visual box size=0.025 0.040 0.065
- link left_wheel: geometry collision cylinder length=0.050 radius=0.050; visual cylinder length=0.050 radius=0.050
- link rear_caster_bracket: geometry collision box size=0.025 0.040 0.065; visual box size=0.025 0.040 0.065
- link right_wheel: geometry collision cylinder length=0.050 radius=0.050; visual cylinder length=0.050 radius=0.050
Joints:
- removed joint base_to_l_motor_brk
- removed joint base_to_post_1
- removed joint base_to_post_2
- removed joint base_to_post_3
- removed joint base_to_post_4
- removed joint base_to_r_motor_brk
- removed joint l_brk_to_l_motor
- removed joint l_brk_to_wheel
- removed joint post_1_to_rear_platform
- removed joint r_brk_to_r_motor
- removed joint r_brk_to_wheel
- added joint base_to_fwd_post_1: type fixed, parent base_link, child fwd_post_1, origin xyz=0.14 0.08 0.005
- added joint base_to_fwd_post_2: type fixed, parent base_link, child fwd_post_2, origin xyz=0.14 -0.08 0.005
- added joint base_to_fwd_post_3: type fixed, parent base_link, child fwd_post_3, origin xyz=0.085 -0.08 0.005
- added joint base_to_fwd_post_4: type fixed, parent base_link, child fwd_post_4, origin xyz=0.085 0.08 0.005
- added joint base_to_left_motor_bracket: type fixed, parent base_link, child left_motor_bracket, origin xyz=0.0 0.091 -0.0291
- added joint base_to_rear_post_1: type fixed, parent base_link, child rear_post_1, origin xyz=-0.06 0.08 0.005
- added joint base_to_rear_post_2: type fixed, parent base_link, child rear_post_2, origin xyz=-0.14 0.08 0.005
- added joint base_to_rear_post_3: type fixed, parent base_link, child rear_post_3, origin xyz=-0.06 -0.08 0.005
- added joint base_to_rear_post_4: type fixed, parent base_link, child rear_post_4, origin xyz=-0.14 -0.08 0.005
- added joint base_to_right_motor_bracket: type fixed, parent base_link, child right_motor_bracket, origin xyz=0.0 -0.091 -0.0291
- added joint fwd_platform_to_lidar: type fixed, parent fwd_platform, child laser, origin xyz=-0.015 0.0 0.0455
- added joint fwd_post_1_to_fwd_platform: type fixed, parent fwd_post_1, child fwd_platform, origin xyz=-0.040 -0.080 0.0565
- added joint left_brk_to_left_motor: type fixed, parent left_motor_bracket, child left_motor, origin xyz=0.0 -0.036 -0.004
- added joint left_brk_to_left_wheel: type continuous, parent left_motor_bracket, child left_wheel, origin xyz=0.0 0.029 -0.0105, axis 0 1 0
- added joint rear_post_1_to_rear_platform: type fixed, parent rear_post_1, child rear_platform, origin xyz=-0.040 -0.080 0.0215
- added joint right_brk_to_right_motor: type fixed, parent right_motor_bracket, child right_motor, origin xyz=0.0 0.036 -0.004
- added joint right_brk_to_right_wheel: type continuous, parent right_motor_bracket, child right_wheel, origin xyz=0.0 -0.029 -0.0105, axis 0 1 0
- joint base_to_AAx10: origin xyz=0.060 0.0 0.0 -> xyz=0.070 0.0 -0.020
- joint base_to_USB_PACK: origin xyz=0.060 0.0 0.008 -> xyz=0.060 0.0 0.015
- joint base_to_front_caster: origin xyz=0.150 0.0 -0.070 -> xyz=0.15 0.0 -0.037
- joint base_to_rear_caster: origin xyz=-0.150 0.0 -0.070 -> xyz=-0.15 0.0 -0.037
- joint display_bracket_to_display: origin xyz=0.003 0.008 0.060 -> xyz=0.0055 0.008 0.060
- joint front_caster_bk_to_ball: origin xyz=0.0 0.0 0.004 -> xyz=0.0 0.0 -0.0325
- joint head_fixing_to_servo_block: origin xyz=0.0 0.0 0.047 -> xyz=0.008 0.0 0.039
- joint head_pan: origin xyz=0.0 0.0 0.025 -> xyz=-0.008 0.0 0.033
- joint head_tilt: limit lower=-1.39626 upper=0.698132 effort=1000.0 velocity=0.5 -> lower=-1.39626 upper=0.5 effort=1000.0 velocity=0.698132
- joint neck_to_head_fixing: origin xyz=0.0 0.0 0.30 -> xyz=0.0 0.0 0.150
- joint rear_caster_bk_to_ball: origin xyz=0.0 0.0 0.004 -> xyz=0.0 0.0 -0.0325
- joint rear_platform_to_neck: origin xyz=-0.070 -0.080 -0.028 -> xyz=-0.030 0.0 0.1205
